Commit message: update tcp

File: polymetis/polymetis/data/franka_panda/panda_arm_tcp.urdf (robot description, URDF)
Before this commit: robot panda, 22 links, 21 joints
Joints:
- joint panda_hand_tcp_joint: origin xyz=0 0 0.203865 rpy=0 0 0 -> xyz=0 0 0.190565 rpy=0 0 0

Commit message: update

File: polymetis/polymetis/data/franka_panda/panda_arm_tcp.urdf (robot description, URDF)
Before this commit: robot panda, 22 links, 21 joints
Joints:
- joint panda_hand_tcp_joint: origin xyz=0 0 0.190565 rpy=0 0 0 -> xyz=0 0 0.210565 rpy=0 0 0

Commit message: update

File: polymetis/polymetis/data/franka_panda/panda_arm_tcp.urdf (robot description, URDF)
Before this commit: robot panda, 22 links, 21 joints
Joints:
- joint panda_hand_tcp_joint: origin xyz=0 0 0.210565 rpy=0 0 0 -> xyz=0 0 0.203865 rpy=0 0 0
