Commit message: test

File: polymetis/polymetis/data/franka_panda/panda_arm.urdf (robot description, URDF)
Before this commit: robot panda, 9 links, 8 joints
Joints:
- joint panda_joint8: origin xyz=0 0 0.107 rpy=0 0 0 -> xyz=0 0 0.203865 rpy=0 0 0

Commit message: updates

File: polymetis/polymetis/data/franka_panda/panda_arm.urdf (robot description, URDF)
Before this commit: robot panda, 9 links, 8 joints
Joints:
- joint panda_joint8: origin xyz=0 0 0.203865 rpy=0 0 0 -> xyz=0 0 0.107 rpy=0 0 0

File: polymetis/polymetis/data/franka_panda/panda_arm_tcp.urdf (robot description, URDF)
Before this commit: robot panda, 22 links, 21 joints
Links:
- link panda_hand: geometry collision mesh filename=meshes/collision/hand.stl; visual mesh filename=meshes/visual/hand.dae
- link panda_leftfinger: geometry collision box size=17.5e-3 15.2e-3 18.5e-3; collision box size=17.5e-3 7e-3 23.5e-3
- link panda_link0: geometry collision mesh filename=meshes/collision/link0.stl; visual mesh filename=meshes/visual/link0.dae
- link panda_link1: geometry collision mesh filename=meshes/collision/link1.stl; visual mesh filename=meshes/visual/link1.dae
- link panda_link2: geometry collision mesh filename=meshes/collision/link2.stl; visual mesh filename=meshes/visual/link2.dae
- link panda_link3: geometry collision mesh filename=meshes/collision/link3.stl; visual mesh filename=meshes/visual/link3.dae
- link panda_link4: geometry collision mesh filename=meshes/collision/link4.stl; visual mesh filename=meshes/visual/link4.dae
- link panda_link5: geometry collision mesh filename=meshes/collision/link5.stl; visual mesh filename=meshes/visual/link5.dae
- link panda_link6: geometry collision mesh filename=meshes/collision/link6.stl; visual mesh filename=meshes/visual/link6.dae
- link panda_link7: geometry collision mesh filename=meshes/collision/link7.stl; visual mesh filename=meshes/visual/link7.dae
- link panda_rightfinger: geometry collision box size=17.5e-3 15.2e-3 18.5e-3; collision box size=17.5e-3 7e-3 23.5e-3

File: polymetis/polymetis/data/franka_panda_robotiq_85/panda_robotiq_85.urdf (robot description, URDF)
Before this commit: robot panda, 21 links, 20 joints
Links:
- link robotiq_2f_85_base: geometry collision mesh filename=meshes/robotiq-2f/collision/base.stl scale=0.001 0.001 0.001; visual mesh filename=meshes/robotiq-2f/visual/base.mtl scale=0.1 0.1 0.1
- link robotiq_2f_85_left_coupler: geometry collision mesh filename=meshes/robotiq-2f/collision/coupler.stl scale=0.001 0.001 0.001; visual mesh filename=meshes/robotiq-2f/visual/coupler.mtl scale=0.1 0.1 0.1
- link robotiq_2f_85_left_driver: geometry collision mesh filename=meshes/robotiq-2f/collision/driver.stl scale=0.001 0.001 0.001; visual mesh filename=meshes/robotiq-2f/visual/driver.mtl scale=0.1 0.1 0.1
- link robotiq_2f_85_left_follower: geometry visual mesh filename=meshes/robotiq-2f/visual/follower.mtl scale=0.1 0.1 0.1
- link robotiq_2f_85_left_spring_link: geometry visual mesh filename=meshes/robotiq-2f/visual/spring_link.mtl scale=0.1 0.1 0.1
- link robotiq_2f_85_right_coupler: geometry collision mesh filename=meshes/robotiq-2f/collision/coupler.stl scale=0.001 0.001 0.001; visual mesh filename=meshes/robotiq-2f/visual/coupler.mtl scale=0.1 0.1 0.1
- link robotiq_2f_85_right_driver: geometry collision mesh filename=meshes/robotiq-2f/collision/driver.stl scale=0.001 0.001 0.001; visual mesh filename=meshes/robotiq-2f/visual/driver.mtl scale=0.1 0.1 0.1
- link robotiq_2f_85_right_follower: geometry collision mesh filename=meshes/robotiq-2f/collision/follower.stl scale=0.001 0.001 0.001; visual mesh filename=meshes/robotiq-2f/visual/follower.mtl scale=0.1 0.1 0.1
- link robotiq_2f_85_right_spring_link: geometry collision mesh filename=meshes/robotiq-2f/collision/spring_link.stl scale=0.001 0.001 0.001; visual mesh filename=meshes/robotiq-2f/visual/spring_link.mtl scale=0.1 0.1 0.1

Commit message: update urdf

File: polymetis/polymetis/data/franka_panda/panda_arm.urdf (robot description, URDF)
Before this commit: robot panda, 9 links, 8 joints
Joints:
- joint panda_joint8: origin xyz=0 0 0.203865 rpy=0 0 0 -> xyz=0 0 0.203865 rpy=0 0 -0.7853981633974483

Commit message: update

File: polymetis/polymetis/data/franka_panda/panda_arm.urdf (robot description, URDF)
Before this commit: robot panda, 9 links, 8 joints
Joints:
- joint panda_joint8: origin xyz=0 0 0.203865 rpy=0 0 -0.7853981633974483 -> xyz=0 0 0.203865 rpy=0 0 0
